Commit message: basic definitions done

File: catkin_ws/src/surveillance_payload_simulator/urdf/surveillance_module.urdf (robot description, URDF)
Before this commit: robot surveillance_module, 5 links, 4 joints
Joints:
- joint mast_head_to_pitch: limit lower=0 upper=1.42 effort=30 velocity=1.0 -> lower=-1.42 upper=1.42 effort=30 velocity=1.0; origin (none) -> xyz=0.5 0 3.65 rpy=0 1.5708 0

Commit message: Added prismatic joint to base and mast

File: catkin_ws/src/surveillance_payload_simulator/urdf/surveillance_module.urdf (robot description, URDF)
Before this commit: robot surveillance_module, 5 links, 4 joints
Joints:
- joint base_to_mast: axis (none) -> 0.0 0.0 1.0; limit (none) -> lower=-1.0 upper=3.0 effort=3.0 velocity=1.0; type fixed -> prismatic

Commit message: w.i.p adding model to gazebo

File: catkin_ws/src/surveillance_payload_simulator/urdf/surveillance_module.urdf (robot description, URDF)
Before this commit: robot surveillance_module, 5 links, 4 joints
Links:
- added link world
- link base_link: geometry collision box size=2.0 2.0 1.0; visual box size=2.0 2.0 1.0
- link camera: geometry collision cylinder length=1.0 radius=0.1; visual cylinder length=1.0 radius=0.1
- link mast: geometry collision cylinder length=5.0 radius=0.2; visual cylinder length=5.0 radius=0.2
- link mast_head: geometry collision box size=0.1 0.1 1.0; collision box size=1.0 0.1 0.1
- link pitch_head: geometry collision cylinder length=0.1 radius=0.1; visual cylinder length=0.1 radius=0.1
Joints:
- added joint fixed: type fixed, parent world, child base_link
